File: _saved_H-bridge.sch (KiCad schematic (older format))
At the start: 11 parts, among them U202 L298HN, U401 OP279

Commit message: Assigning footprints
Parts:
- U401: footprint (none) -> Package_SO:TSSOP-8_4.4x3mm_P0.65mm
Changed lines of the file:
@@
 AR Path="/5BEEC4C8/5BE42F54" Ref="U402"  Part="1"
 AR Path="/5BEEC636/5BE42F54" Ref="U502"  Part="1"
-F 0 "U202" H 5650 3550 50  0000 C CNN
+F 0 "U502" H 5650 3550 50  0000 C CNN
 F 1 "L298HN" H 5650 3450 50  0000 C CNN
 F 2 "Package_TO_SOT_THT:TO-220-15_P2.54x2.54mm_StaggerOdd_Lead4.58mm_Vertical" H 5700 2850 50  0001 L CNN
@@
 AR Path="/5BEEC4C8/5BE42F5B" Ref="#PWR0127"  Part="1"
 AR Path="/5BEEC636/5BE42F5B" Ref="#PWR0146"  Part="1"
-F 0 "#PWR0105" H 5650 3950 50  0001 C CNN
+F 0 "#PWR0146" H 5650 3950 50  0001 C CNN
 F 1 "GND" H 5655 4027 50  0000 C CNN
 F 2 "" H 5650 4200 50  0001 C CNN
@@
 AR Path="/5BEEC4C8/5BE42F71" Ref="R406"  Part="1"
 AR Path="/5BEEC636/5BE42F71" Ref="R506"  Part="1"
-F 0 "R206" H 5520 4696 50  0000 L CNN
+F 0 "R506" H 5520 4696 50  0000 L CNN
 F 1 "200mR" H 5520 4605 50  0000 L CNN
 F 2 "Resistor_SMD:R_0805_2012Metric" V 5380 4650 50  0001 C CNN
@@
 AR Path="/5BEEC4C8/5BE42F78" Ref="#PWR0128"  Part="1"
 AR Path="/5BEEC636/5BE42F78" Ref="#PWR0147"  Part="1"
-F 0 "#PWR0106" H 5450 4550 50  0001 C CNN
+F 0 "#PWR0147" H 5450 4550 50  0001 C CNN
 F 1 "GND" H 5455 4627 50  0000 C CNN
 F 2 "" H 5450 4800 50  0001 C CNN
@@
 AR Path="/5BEEC4C8/5BE42F8D" Ref="C401"  Part="1"
 AR Path="/5BEEC636/5BE42F8D" Ref="C501"  Part="1"
-F 0 "C201" V 4398 2650 50  0000 C CNN
+F 0 "C501" V 4398 2650 50  0000 C CNN
 F 1 "100nF" V 4489 2650 50  0000 C CNN
 F 2 "Capacitor_SMD:C_0805_2012Metric" H 4688 2500 50  0001 C CNN
@@
 AR Path="/5BEEC4C8/5BE42F94" Ref="C403"  Part="1"
 AR Path="/5BEEC636/5BE42F94" Ref="C503"  Part="1"
-F 0 "C203" V 6148 2650 50  0000 C CNN
+F 0 "C503" V 6148 2650 50  0000 C CNN
 F 1 "100nF" V 6239 2650 50  0000 C CNN
 F 2 "Capacitor_SMD:C_0805_2012Metric" H 6438 2500 50  0001 C CNN
@@
 AR Path="/5BEEC4C8/5BE42FA7" Ref="#PWR0129"  Part="1"
 AR Path="/5BEEC636/5BE42FA7" Ref="#PWR0148"  Part="1"
-F 0 "#PWR0107" H 4650 2550 50  0001 C CNN
+F 0 "#PWR0148" H 4650 2550 50  0001 C CNN
 F 1 "GND" H 4655 2627 50  0000 C CNN
 F 2 "" H 4650 2800 50  0001 C CNN
@@
 AR Path="/5BEEC4C8/5BE4772A" Ref="R405"  Part="1"
 AR Path="/5BEEC636/5BE4772A" Ref="R505"  Part="1"
-F 0 "R205" H 5200 4700 50  0000 L CNN
+F 0 "R505" H 5200 4700 50  0000 L CNN
 F 1 "200mR" H 5000 4600 50  0000 L CNN
 F 2 "Resistor_SMD:R_0805_2012Metric" V 5280 4650 50  0001 C CNN
@@
 AR Path="/5BEEC4C8/5BE47731" Ref="#PWR0130"  Part="1"
 AR Path="/5BEEC636/5BE47731" Ref="#PWR0149"  Part="1"
-F 0 "#PWR0108" H 5350 4550 50  0001 C CNN
+F 0 "#PWR0149" H 5350 4550 50  0001 C CNN
 F 1 "GND" H 5355 4627 50  0000 C CNN
 F 2 "" H 5350 4800 50  0001 C CNN
@@
 AR Path="/5BEEC4C8/5BEE040B" Ref="#PWR0131"  Part="1"
 AR Path="/5BEEC636/5BEE040B" Ref="#PWR0150"  Part="1"
-F 0 "#PWR0109" H 6400 2550 50  0001 C CNN
+F 0 "#PWR0150" H 6400 2550 50  0001 C CNN
 F 1 "GND" H 6405 2627 50  0000 C CNN
 F 2 "" H 6400 2800 50  0001 C CNN
@@
 AR Path="/5BEEC4C8/5BEE8828" Ref="#PWR0132"  Part="1"
 AR Path="/5BEEC636/5BEE8828" Ref="#PWR0151"  Part="1"
-F 0 "#PWR0110" H 6400 2350 50  0001 C CNN
+F 0 "#PWR0151" H 6400 2350 50  0001 C CNN
 F 1 "+12V" H 6415 2673 50  0000 C CNN
 F 2 "" H 6400 2500 50  0001 C CNN
@@
 AR Path="/5BEEC4C8/5BEEBB70" Ref="#PWR0141"  Part="1"
 AR Path="/5BEEC636/5BEEBB70" Ref="#PWR0160"  Part="1"
-F 0 "#PWR0119" H 4550 2350 50  0001 C CNN
+F 0 "#PWR0160" H 4550 2350 50  0001 C CNN
 F 1 "+5V" H 4565 2673 50  0000 C CNN
 F 2 "" H 4550 2500 50  0001 C CNN
@@
 AR Path="/5BEEC4C8/5C4B589F" Ref="R401"  Part="1"
 AR Path="/5BEEC636/5C4B589F" Ref="R501"  Part="1"
-F 0 "R201" V 4200 4750 50  0000 R CNN
+F 0 "R501" V 4200 4750 50  0000 R CNN
 F 1 "1k" V 4400 4750 50  0000 R CNN
 F 2 "Resistor_SMD:R_0805_2012Metric" V 4230 4700 50  0001 C CNN
@@
 AR Path="/5BEEC4C8/5C4B6CEE" Ref="#PWR0143"  Part="1"
 AR Path="/5BEEC636/5C4B6CEE" Ref="#PWR0162"  Part="1"
-F 0 "#PWR0121" H 5500 5900 50  0001 C CNN
+F 0 "#PWR0162" H 5500 5900 50  0001 C CNN
 F 1 "+5V" H 5515 6223 50  0000 C CNN
 F 2 "" H 5500 6050 50  0001 C CNN
@@
 AR Path="/5BEEC4C8/5C4B6D58" Ref="C402"  Part="1"
 AR Path="/5BEEC636/5C4B6D58" Ref="C502"  Part="1"
-F 0 "C202" H 6065 6396 50  0000 L CNN
+F 0 "C502" H 6065 6396 50  0000 L CNN
 F 1 "100nF" H 6065 6305 50  0000 L CNN
 F 2 "Capacitor_SMD:C_0805_2012Metric" H 5988 6200 50  0001 C CNN
@@
 AR Path="/5BEEC4C8/5C4B6E7F" Ref="#PWR0144"  Part="1"
 AR Path="/5BEEC636/5C4B6E7F" Ref="#PWR0163"  Part="1"
-F 0 "#PWR0122" H 5500 6400 50  0001 C CNN
+F 0 "#PWR0163" H 5500 6400 50  0001 C CNN
 F 1 "GND" H 5505 6477 50  0000 C CNN
 F 2 "" H 5500 6650 50  0001 C CNN
@@
 AR Path="/5BEEC4C8/5C4B7865" Ref="#PWR0145"  Part="1"
 AR Path="/5BEEC636/5C4B7865" Ref="#PWR0164"  Part="1"
-F 0 "#PWR0123" H 4650 4800 50  0001 C CNN
+F 0 "#PWR0164" H 4650 4800 50  0001 C CNN
 F 1 "GND" H 4655 4877 50  0000 C CNN
 F 2 "" H 4650 5050 50  0001 C CNN
@@
 AR Path="/5BEEC636/5C5CDC2F" Ref="U501"  Part="1"
 AR Path="/5BE41DDF/5C5CDC2F" Ref="U201"  Part="1"
-F 0 "U201" H 4350 4817 50  0000 C CNN
+F 0 "U501" H 4350 4817 50  0000 C CNN
 F 1 "OP279" H 4350 4726 50  0000 C CNN
-F 2 "" H 4350 4450 50  0001 C CNN
+F 2 "Package_SO:TSSOP-8_4.4x3mm_P0.65mm" H 4350 4450 50  0001 C CNN
 F 3 "http://www.analog.com/media/en/technical-documentation/data-sheets/OP179_279.pdf" H 4350 4450 50  0001 C CNN
 	1    4350 4450
@@
 AR Path="/5BEEC636/5C5CE16B" Ref="U501"  Part="2"
 AR Path="/5BE41DDF/5C5CE16B" Ref="U201"  Part="2"
-F 0 "U201" H 4350 5917 50  0000 C CNN
+F 0 "U501" H 4350 5917 50  0000 C CNN
 F 1 "OP279" H 4350 5826 50  0000 C CNN
-F 2 "" H 4350 5550 50  0001 C CNN
+F 2 "Package_SO:TSSOP-8_4.4x3mm_P0.65mm" H 4350 5550 50  0001 C CNN
 F 3 "http://www.analog.com/media/en/technical-documentation/data-sheets/OP179_279.pdf" H 4350 5550 50  0001 C CNN
 	2    4350 5550
@@
 AR Path="/5BEEC636/5C5CE212" Ref="U501"  Part="3"
 AR Path="/5BE41DDF/5C5CE212" Ref="U201"  Part="3"
-F 0 "U201" H 5558 6396 50  0000 L CNN
+F 0 "U501" H 5558 6396 50  0000 L CNN
 F 1 "OP279" H 5558 6305 50  0000 L CNN
-F 2 "" H 5600 6350 50  0001 C CNN
+F 2 "Package_SO:TSSOP-8_4.4x3mm_P0.65mm" H 5600 6350 50  0001 C CNN
 F 3 "http://www.analog.com/media/en/technical-documentation/data-sheets/OP179_279.pdf" H 5600 6350 50  0001 C CNN
 	3    5600 6350
@@
 AR Path="/5BEEC4C8/5C5D032D" Ref="R403"  Part="1"
 AR Path="/5BEEC636/5C5D032D" Ref="R503"  Part="1"
-F 0 "R203" V 4550 4950 50  0000 R CNN
+F 0 "R503" V 4550 4950 50  0000 R CNN
 F 1 "10k" V 4750 4950 50  0000 R CNN
 F 2 "Resistor_SMD:R_0805_2012Metric" V 4580 4900 50  0001 C CNN
@@
 AR Path="/5BEEC4C8/5C5D589D" Ref="R402"  Part="1"
 AR Path="/5BEEC636/5C5D589D" Ref="R502"  Part="1"
-F 0 "R202" V 4200 5850 50  0000 R CNN
+F 0 "R502" V 4200 5850 50  0000 R CNN
 F 1 "1k" V 4400 5850 50  0000 R CNN
 F 2 "Resistor_SMD:R_0805_2012Metric" V 4230 5800 50  0001 C CNN
@@
 AR Path="/5BEEC4C8/5C5D58A6" Ref="#PWR0154"  Part="1"
 AR Path="/5BEEC636/5C5D58A6" Ref="#PWR0156"  Part="1"
-F 0 "#PWR0152" H 4650 5900 50  0001 C CNN
+F 0 "#PWR0156" H 4650 5900 50  0001 C CNN
 F 1 "GND" H 4655 5977 50  0000 C CNN
 F 2 "" H 4650 6150 50  0001 C CNN
@@
 AR Path="/5BEEC4C8/5C5D58B3" Ref="R404"  Part="1"
 AR Path="/5BEEC636/5C5D58B3" Ref="R504"  Part="1"
-F 0 "R204" V 4550 6050 50  0000 R CNN
+F 0 "R504" V 4550 6050 50  0000 R CNN
 F 1 "10k" V 4750 6050 50  0000 R CNN
 F 2 "Resistor_SMD:R_0805_2012Metric" V 4580 6000 50  0001 C CNN
@@
 AR Path="/5BEEC4C8/5C5EBA06" Ref="#PWR0155"  Part="1"
 AR Path="/5BEEC636/5C5EBA06" Ref="#PWR0157"  Part="1"
-F 0 "#PWR0153" H 4400 3050 50  0001 C CNN
+F 0 "#PWR0157" H 4400 3050 50  0001 C CNN
 F 1 "+5V" H 4415 3373 50  0000 C CNN
 F 2 "" H 4400 3200 50  0001 C CNN
