File: _saved_Mars Rover.sch (KiCad schematic (older format))
At the start: 21 parts, among them J1 Barrel_Jack, J101 Conn_01x02, J102 Conn_01x03, J103 Conn_01x03, J104 Conn_01x03, J105 Conn_01x03, J106 Conn_01x03, J107 Conn_01x03, J108 Conn_01x03, J109 Conn_01x01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

Commit message: Assigning footprints
Parts:
- H102, H103, H104, H105, H106: footprint MountingHole:MountingHole_2.7mm -> (none)
- SW1, SW101: footprint (none) -> Connector_PinHeader_2.54mm:PinHeader_1x02_P2.54mm_Vertical
- U101: footprint (none) -> Package_SO:TSSOP-20_4.4x6.5mm_P0.65mm
Changed lines of the file:
@@
 F 0 "SW1" H 1900 2485 50  0000 C CNN
 F 1 "KILLSWITCH" H 1900 2394 50  0000 C CNN
-F 2 "" H 1900 2250 50  0001 C CNN
+F 2 "Connector_PinHeader_2.54mm:PinHeader_1x02_P2.54mm_Vertical" H 1900 2250 50  0001 C CNN
 F 3 "" H 1900 2250 50  0001 C CNN
 	1    1900 2250
@@
 F 1 "Barrel_Jack" H 1255 2584 50  0000 C CNN
 F 2 "Connector_BarrelJack:BarrelJack_CUI_PJ-102AH_Horizontal" H 1250 2310 50  0001 C CNN
-F 3 "~" H 1250 2310 50  0001 C CNN
+F 3 "CONFIRM FOOTPRINT" H 1250 2310 50  0001 C CNN
 	1    1200 2350
 	1    0    0    -1
@@
 F 0 "SW101" H 5750 2485 50  0000 C CNN
 F 1 "CHARGING" H 5750 2394 50  0000 C CNN
-F 2 "" H 5750 2250 50  0001 C CNN
+F 2 "Connector_PinHeader_2.54mm:PinHeader_1x02_P2.54mm_Vertical" H 5750 2250 50  0001 C CNN
 F 3 "" H 5750 2250 50  0001 C CNN
 	1    5750 2250
@@
 F 0 "H102" H 9950 3196 50  0000 L CNN
 F 1 "MountingHole" H 9950 3105 50  0000 L CNN
-F 2 "MountingHole:MountingHole_2.7mm" H 9850 3150 50  0001 C CNN
+F 2 "" H 9850 3150 50  0001 C CNN
 F 3 "~" H 9850 3150 50  0001 C CNN
 	1    9850 3150
@@
 F 0 "H103" H 9950 3446 50  0000 L CNN
 F 1 "MountingHole" H 9950 3355 50  0000 L CNN
-F 2 "MountingHole:MountingHole_2.7mm" H 9850 3400 50  0001 C CNN
+F 2 "" H 9850 3400 50  0001 C CNN
 F 3 "~" H 9850 3400 50  0001 C CNN
 	1    9850 3400
@@
 F 0 "H104" H 9950 3696 50  0000 L CNN
 F 1 "MountingHole" H 9950 3605 50  0000 L CNN
-F 2 "MountingHole:MountingHole_2.7mm" H 9850 3650 50  0001 C CNN
+F 2 "" H 9850 3650 50  0001 C CNN
 F 3 "~" H 9850 3650 50  0001 C CNN
 	1    9850 3650
@@
 F 0 "H105" H 9950 3946 50  0000 L CNN
 F 1 "MountingHole" H 9950 3855 50  0000 L CNN
-F 2 "MountingHole:MountingHole_2.7mm" H 9850 3900 50  0001 C CNN
+F 2 "" H 9850 3900 50  0001 C CNN
 F 3 "~" H 9850 3900 50  0001 C CNN
 	1    9850 3900
@@
 F 0 "H106" H 9950 4196 50  0000 L CNN
 F 1 "MountingHole" H 9950 4105 50  0000 L CNN
-F 2 "MountingHole:MountingHole_2.7mm" H 9850 4150 50  0001 C CNN
+F 2 "" H 9850 4150 50  0001 C CNN
 F 3 "~" H 9850 4150 50  0001 C CNN
 	1    9850 4150
@@
 F 0 "U101" H 3200 5500 50  0000 C CNN
 F 1 "74HCT244" H 3200 5400 50  0000 C CNN
-F 2 "" H 3450 4700 50  0001 C CNN
+F 2 "Package_SO:TSSOP-20_4.4x6.5mm_P0.65mm" H 3450 4700 50  0001 C CNN
 F 3 "http://www.nxp.com/documents/data_sheet/74HC_HCT244.pdf" H 3450 4700 50  0001 C CNN
 	1    3450 4700
