File: _saved_digital.sch (KiCad schematic (older format))
At the start: 9 parts, among them J1401 Raspberry_Pi_2_3, U1401 PCA9685PW, U1402 ADS7828, U1403 Rpi0w

Commit message: Assigning footprints
Parts:
- U1403: footprint (none) -> Roverschemlib:raspi0w
Changed lines of the file:
@@
 F 0 "U1403" H 9150 3897 60  0000 C CNN
 F 1 "Rpi0w" H 9150 3791 60  0000 C CNN
-F 2 "" H 9150 1500 60  0001 C CNN
+F 2 "Roverschemlib:raspi0w" H 9150 1500 60  0001 C CNN
 F 3 "" H 9150 1500 60  0001 C CNN
 	1    9150 1500
