File: Mars Rover.sch (KiCad schematic (older format))
At the start: 21 parts, among them J1 Barrel_Jack, J101 Conn_01x02, J102 Conn_01x03, J103 Conn_01x03, J104 Conn_01x03, J105 Conn_01x03, J106 Conn_01x03, J107 Conn_01x03, J108 Conn_01x03, J109 Conn_01x01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

Commit message: Schematics done, now assigning footprints to do PCB Next
Parts:
- C101, C102: footprint (none) -> Capacitor_SMD:C_0805_2012Metric
- H102, H103, H104, H105, H106: footprint (none) -> MountingHole:MountingHole_2.7mm
- J1: footprint (none) -> Connector_BarrelJack:BarrelJack_CUI_PJ-102AH_Horizontal
Changed lines of the file:
@@
 F 0 "J1" H 1255 2675 50  0000 C CNN
 F 1 "Barrel_Jack" H 1255 2584 50  0000 C CNN
-F 2 "" H 1250 2310 50  0001 C CNN
+F 2 "Connector_BarrelJack:BarrelJack_CUI_PJ-102AH_Horizontal" H 1250 2310 50  0001 C CNN
 F 3 "~" H 1250 2310 50  0001 C CNN
 	1    1200 2350
@@
 F 0 "C101" H 1365 2896 50  0000 L CNN
 F 1 "22uF" H 1365 2805 50  0000 L CNN
-F 2 "" H 1250 2850 50  0001 C CNN
+F 2 "Capacitor_SMD:C_0805_2012Metric" H 1250 2850 50  0001 C CNN
 F 3 "~" H 1250 2850 50  0001 C CNN
 	1    1250 2850
@@
 F 0 "C102" H 1485 2804 50  0000 R CNN
 F 1 "0.1uF" H 1485 2895 50  0000 R CNN
-F 2 "" H 1638 2700 50  0001 C CNN
+F 2 "Capacitor_SMD:C_0805_2012Metric" H 1638 2700 50  0001 C CNN
 F 3 "~" H 1600 2850 50  0001 C CNN
 	1    1600 2850
@@
 F 0 "H102" H 9950 3196 50  0000 L CNN
 F 1 "MountingHole" H 9950 3105 50  0000 L CNN
-F 2 "" H 9850 3150 50  0001 C CNN
+F 2 "MountingHole:MountingHole_2.7mm" H 9850 3150 50  0001 C CNN
 F 3 "~" H 9850 3150 50  0001 C CNN
 	1    9850 3150
@@
 F 0 "H103" H 9950 3446 50  0000 L CNN
 F 1 "MountingHole" H 9950 3355 50  0000 L CNN
-F 2 "" H 9850 3400 50  0001 C CNN
+F 2 "MountingHole:MountingHole_2.7mm" H 9850 3400 50  0001 C CNN
 F 3 "~" H 9850 3400 50  0001 C CNN
 	1    9850 3400
@@
 F 0 "H104" H 9950 3696 50  0000 L CNN
 F 1 "MountingHole" H 9950 3605 50  0000 L CNN
-F 2 "" H 9850 3650 50  0001 C CNN
+F 2 "MountingHole:MountingHole_2.7mm" H 9850 3650 50  0001 C CNN
 F 3 "~" H 9850 3650 50  0001 C CNN
 	1    9850 3650
@@
 F 0 "H105" H 9950 3946 50  0000 L CNN
 F 1 "MountingHole" H 9950 3855 50  0000 L CNN
-F 2 "" H 9850 3900 50  0001 C CNN
+F 2 "MountingHole:MountingHole_2.7mm" H 9850 3900 50  0001 C CNN
 F 3 "~" H 9850 3900 50  0001 C CNN
 	1    9850 3900
@@
 F 0 "H106" H 9950 4196 50  0000 L CNN
 F 1 "MountingHole" H 9950 4105 50  0000 L CNN
-F 2 "" H 9850 4150 50  0001 C CNN
+F 2 "MountingHole:MountingHole_2.7mm" H 9850 4150 50  0001 C CNN
 F 3 "~" H 9850 4150 50  0001 C CNN
 	1    9850 4150

Commit message: Assigning footprints
Parts:
- U101: footprint (none) -> Package_SO:TSSOP-20_4.4x6.5mm_P0.65mm
Changed lines of the file:
@@
 F 0 "U101" H 3200 5500 50  0000 C CNN
 F 1 "74HCT244" H 3200 5400 50  0000 C CNN
-F 2 "" H 3450 4700 50  0001 C CNN
+F 2 "Package_SO:TSSOP-20_4.4x6.5mm_P0.65mm" H 3450 4700 50  0001 C CNN
 F 3 "http://www.nxp.com/documents/data_sheet/74HC_HCT244.pdf" H 3450 4700 50  0001 C CNN
 	1    3450 4700

Commit message: on to pcbs
Parts:
- H101: footprint (none) -> MountingHole:MountingHole_3.2mm_M3_Pad
- H102, H103, H104, H105, H106: footprint MountingHole:MountingHole_2.7mm -> MountingHole:MountingHole_3.2mm_M3
- J101, SW1, SW101: footprint (none) -> Connector_PinHeader_2.54mm:PinHeader_1x02_P2.54mm_Vertical
- J102, J103, J104, J105, J106, J107, J108: footprint (none) -> Connector_PinHeader_2.54mm:PinHeader_1x03_P2.54mm_Vertical_SMD_Pin1Right
- J109: footprint (none) -> Connector_PinHeader_2.54mm:PinHeader_1x01_P2.54mm_Horizontal
Changed lines of the file:
@@
 F 0 "SW1" H 1900 2485 50  0000 C CNN
 F 1 "KILLSWITCH" H 1900 2394 50  0000 C CNN
-F 2 "" H 1900 2250 50  0001 C CNN
+F 2 "Connector_PinHeader_2.54mm:PinHeader_1x02_P2.54mm_Vertical" H 1900 2250 50  0001 C CNN
 F 3 "" H 1900 2250 50  0001 C CNN
 	1    1900 2250
@@
 F 1 "Barrel_Jack" H 1255 2584 50  0000 C CNN
 F 2 "Connector_BarrelJack:BarrelJack_CUI_PJ-102AH_Horizontal" H 1250 2310 50  0001 C CNN
-F 3 "~" H 1250 2310 50  0001 C CNN
+F 3 "CONFIRM FOOTPRINT" H 1250 2310 50  0001 C CNN
 	1    1200 2350
 	1    0    0    -1
@@
 F 0 "SW101" H 5750 2485 50  0000 C CNN
 F 1 "CHARGING" H 5750 2394 50  0000 C CNN
-F 2 "" H 5750 2250 50  0001 C CNN
+F 2 "Connector_PinHeader_2.54mm:PinHeader_1x02_P2.54mm_Vertical" H 5750 2250 50  0001 C CNN
 F 3 "" H 5750 2250 50  0001 C CNN
 	1    5750 2250
@@
 F 0 "J101" H 720 2475 50  0000 C CNN
 F 1 "Conn_01x02" H 720 2566 50  0000 C CNN
-F 2 "" H 800 2800 50  0001 C CNN
+F 2 "Connector_PinHeader_2.54mm:PinHeader_1x02_P2.54mm_Vertical" H 800 2800 50  0001 C CNN
 F 3 "~" H 800 2800 50  0001 C CNN
 	1    800  2800
@@
 F 0 "J109" H 1770 2375 50  0000 C CNN
 F 1 "Conn_01x01" H 1770 2466 50  0000 C CNN
-F 2 "" H 1850 2600 50  0001 C CNN
+F 2 "Connector_PinHeader_2.54mm:PinHeader_1x01_P2.54mm_Horizontal" H 1850 2600 50  0001 C CNN
 F 3 "~" H 1850 2600 50  0001 C CNN
 	1    1850 2600
@@
 F 0 "H101" H 9950 2651 50  0000 L CNN
 F 1 "MountingHole_Pad" H 9950 2560 50  0000 L CNN
-F 2 "" H 9850 2600 50  0001 C CNN
+F 2 "MountingHole:MountingHole_3.2mm_M3_Pad" H 9850 2600 50  0001 C CNN
 F 3 "~" H 9850 2600 50  0001 C CNN
 	1    9850 2600
@@
 F 0 "H102" H 9950 3196 50  0000 L CNN
 F 1 "MountingHole" H 9950 3105 50  0000 L CNN
-F 2 "MountingHole:MountingHole_2.7mm" H 9850 3150 50  0001 C CNN
+F 2 "MountingHole:MountingHole_3.2mm_M3" H 9850 3150 50  0001 C CNN
 F 3 "~" H 9850 3150 50  0001 C CNN
 	1    9850 3150
@@
 F 0 "H103" H 9950 3446 50  0000 L CNN
 F 1 "MountingHole" H 9950 3355 50  0000 L CNN
-F 2 "MountingHole:MountingHole_2.7mm" H 9850 3400 50  0001 C CNN
+F 2 "MountingHole:MountingHole_3.2mm_M3" H 9850 3400 50  0001 C CNN
 F 3 "~" H 9850 3400 50  0001 C CNN
 	1    9850 3400
@@
 F 0 "H104" H 9950 3696 50  0000 L CNN
 F 1 "MountingHole" H 9950 3605 50  0000 L CNN
-F 2 "MountingHole:MountingHole_2.7mm" H 9850 3650 50  0001 C CNN
+F 2 "MountingHole:MountingHole_3.2mm_M3" H 9850 3650 50  0001 C CNN
 F 3 "~" H 9850 3650 50  0001 C CNN
 	1    9850 3650
@@
 F 0 "H105" H 9950 3946 50  0000 L CNN
 F 1 "MountingHole" H 9950 3855 50  0000 L CNN
-F 2 "MountingHole:MountingHole_2.7mm" H 9850 3900 50  0001 C CNN
+F 2 "MountingHole:MountingHole_3.2mm_M3" H 9850 3900 50  0001 C CNN
 F 3 "~" H 9850 3900 50  0001 C CNN
 	1    9850 3900
@@
 F 0 "H106" H 9950 4196 50  0000 L CNN
 F 1 "MountingHole" H 9950 4105 50  0000 L CNN
-F 2 "MountingHole:MountingHole_2.7mm" H 9850 4150 50  0001 C CNN
+F 2 "MountingHole:MountingHole_3.2mm_M3" H 9850 4150 50  0001 C CNN
 F 3 "~" H 9850 4150 50  0001 C CNN
 	1    9850 4150
@@
 F 0 "J103" H 970 3875 50  0000 C CNN
 F 1 "Conn_01x03" H 970 3966 50  0000 C CNN
-F 2 "" H 1050 4200 50  0001 C CNN
+F 2 "Connector_PinHeader_2.54mm:PinHeader_1x03_P2.54mm_Vertical_SMD_Pin1Right" H 1050 4200 50  0001 C CNN
 F 3 "~" H 1050 4200 50  0001 C CNN
 	1    1050 4200
@@
 F 0 "J104" V 1250 4650 50  0000 C CNN
 F 1 "Conn_01x03" V 1150 4650 50  0000 C CNN
-F 2 "" H 1050 4650 50  0001 C CNN
+F 2 "Connector_PinHeader_2.54mm:PinHeader_1x03_P2.54mm_Vertical_SMD_Pin1Right" H 1050 4650 50  0001 C CNN
 F 3 "~" H 1050 4650 50  0001 C CNN
 	1    1050 4650
@@
 F 0 "J105" V 1250 5100 50  0000 C CNN
 F 1 "Conn_01x03" V 1150 5100 50  0000 C CNN
-F 2 "" H 1050 5100 50  0001 C CNN
+F 2 "Connector_PinHeader_2.54mm:PinHeader_1x03_P2.54mm_Vertical_SMD_Pin1Right" H 1050 5100 50  0001 C CNN
 F 3 "~" H 1050 5100 50  0001 C CNN
 	1    1050 5100
@@
 F 0 "J106" V 1300 5550 50  0000 C CNN
 F 1 "Conn_01x03" V 1200 5550 50  0000 C CNN
-F 2 "" H 1050 5550 50  0001 C CNN
+F 2 "Connector_PinHeader_2.54mm:PinHeader_1x03_P2.54mm_Vertical_SMD_Pin1Right" H 1050 5550 50  0001 C CNN
 F 3 "~" H 1050 5550 50  0001 C CNN
 	1    1050 5550
@@
 F 0 "J107" V 1300 6050 50  0000 C CNN
 F 1 "Conn_01x03" V 1200 6050 50  0000 C CNN
-F 2 "" H 1050 6050 50  0001 C CNN
+F 2 "Connector_PinHeader_2.54mm:PinHeader_1x03_P2.54mm_Vertical_SMD_Pin1Right" H 1050 6050 50  0001 C CNN
 F 3 "~" H 1050 6050 50  0001 C CNN
 	1    1050 6050
@@
 F 0 "J108" V 1300 6450 50  0000 C CNN
 F 1 "Conn_01x03" V 1200 6450 50  0000 C CNN
-F 2 "" H 1050 6450 50  0001 C CNN
+F 2 "Connector_PinHeader_2.54mm:PinHeader_1x03_P2.54mm_Vertical_SMD_Pin1Right" H 1050 6450 50  0001 C CNN
 F 3 "~" H 1050 6450 50  0001 C CNN
 	1    1050 6450
@@
 F 0 "J102" V 1250 6850 50  0000 C CNN
 F 1 "Conn_01x03" V 1150 6850 50  0000 C CNN
-F 2 "" H 1000 6850 50  0001 C CNN
+F 2 "Connector_PinHeader_2.54mm:PinHeader_1x03_P2.54mm_Vertical_SMD_Pin1Right" H 1000 6850 50  0001 C CNN
 F 3 "~" H 1000 6850 50  0001 C CNN
 	1    1000 6850
