File: Mars Rover.sch (KiCad schematic (older format))
At the start: 21 parts, among them J1 Barrel_Jack, J101 Conn_01x02, J102 Conn_01x03, J103 Conn_01x03, J104 Conn_01x03, J105 Conn_01x03, J106 Conn_01x03, J107 Conn_01x03, J108 Conn_01x03, J109 Conn_01x01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

Commit message: updated layout
Parts:
- added J110: Conn_01x03, Connector_PinHeader_2.54mm:PinHeader_1x03_P2.54mm_Vertical, symbol Connector_Generic:Conn_01x03
- J102, J103, J104, J105, J106, J107, J108: footprint Connector_PinHeader_2.54mm:PinHeader_1x03_P2.54mm_Vertical_SMD_Pin1Right -> Connector_PinHeader_2.54mm:PinHeader_1x03_P2.54mm_Vertical
Connections:
- net +7.5V: now also J110.3 (Pin_3)
- net Digital logic/PWMD: now also U101.11 (2A3)
- net GND: now also J110.1 (Pin_1); no longer U101.1 (1OE)
- net at U101.9 (2Y3): now also J110.2 (Pin_2)
- no-connect marks 2 -> 0
Other:
- moved on the sheet: J102
Changed lines of the file:
@@
 F13 "PWMB" I L 4150 4700 50
 F14 "PWMC" I L 4150 4800 50
-F15 "PWMD" I L 4150 3200 50
+F15 "PWMD" I L 4150 4900 50
 F16 "PWME" I L 4150 3300 50
 F17 "PWMF" I L 4150 3400 50
@@
 F 0 "J103" H 970 3875 50  0000 C CNN
 F 1 "Conn_01x03" H 970 3966 50  0000 C CNN
-F 2 "Connector_PinHeader_2.54mm:PinHeader_1x03_P2.54mm_Vertical_SMD_Pin1Right" H 1050 4200 50  0001 C CNN
+F 2 "Connector_PinHeader_2.54mm:PinHeader_1x03_P2.54mm_Vertical" H 1050 4200 50  0001 C CNN
 F 3 "~" H 1050 4200 50  0001 C CNN
 	1    1050 4200
@@
 F 0 "J104" V 1250 4650 50  0000 C CNN
 F 1 "Conn_01x03" V 1150 4650 50  0000 C CNN
-F 2 "Connector_PinHeader_2.54mm:PinHeader_1x03_P2.54mm_Vertical_SMD_Pin1Right" H 1050 4650 50  0001 C CNN
+F 2 "Connector_PinHeader_2.54mm:PinHeader_1x03_P2.54mm_Vertical" H 1050 4650 50  0001 C CNN
 F 3 "~" H 1050 4650 50  0001 C CNN
 	1    1050 4650
@@
 F 0 "J105" V 1250 5100 50  0000 C CNN
 F 1 "Conn_01x03" V 1150 5100 50  0000 C CNN
-F 2 "Connector_PinHeader_2.54mm:PinHeader_1x03_P2.54mm_Vertical_SMD_Pin1Right" H 1050 5100 50  0001 C CNN
+F 2 "Connector_PinHeader_2.54mm:PinHeader_1x03_P2.54mm_Vertical" H 1050 5100 50  0001 C CNN
 F 3 "~" H 1050 5100 50  0001 C CNN
 	1    1050 5100
@@
 F 0 "J106" V 1300 5550 50  0000 C CNN
 F 1 "Conn_01x03" V 1200 5550 50  0000 C CNN
-F 2 "Connector_PinHeader_2.54mm:PinHeader_1x03_P2.54mm_Vertical_SMD_Pin1Right" H 1050 5550 50  0001 C CNN
+F 2 "Connector_PinHeader_2.54mm:PinHeader_1x03_P2.54mm_Vertical" H 1050 5550 50  0001 C CNN
 F 3 "~" H 1050 5550 50  0001 C CNN
 	1    1050 5550
@@
 F 0 "J107" V 1300 6050 50  0000 C CNN
 F 1 "Conn_01x03" V 1200 6050 50  0000 C CNN
-F 2 "Connector_PinHeader_2.54mm:PinHeader_1x03_P2.54mm_Vertical_SMD_Pin1Right" H 1050 6050 50  0001 C CNN
+F 2 "Connector_PinHeader_2.54mm:PinHeader_1x03_P2.54mm_Vertical" H 1050 6050 50  0001 C CNN
 F 3 "~" H 1050 6050 50  0001 C CNN
 	1    1050 6050
@@
 F 0 "J108" V 1300 6450 50  0000 C CNN
 F 1 "Conn_01x03" V 1200 6450 50  0000 C CNN
-F 2 "Connector_PinHeader_2.54mm:PinHeader_1x03_P2.54mm_Vertical_SMD_Pin1Right" H 1050 6450 50  0001 C CNN
+F 2 "Connector_PinHeader_2.54mm:PinHeader_1x03_P2.54mm_Vertical" H 1050 6450 50  0001 C CNN
 F 3 "~" H 1050 6450 50  0001 C CNN
 	1    1050 6450
@@
 L Connector_Generic:Conn_01x03 J102
 U 1 1 5C591EF2
-P 1000 6850
-F 0 "J102" V 1250 6850 50  0000 C CNN
-F 1 "Conn_01x03" V 1150 6850 50  0000 C CNN
-F 2 "Connector_PinHeader_2.54mm:PinHeader_1x03_P2.54mm_Vertical_SMD_Pin1Right" H 1000 6850 50  0001 C CNN
-F 3 "~" H 1000 6850 50  0001 C CNN
-	1    1000 6850
+P 1050 6850
+F 0 "J102" V 1300 6850 50  0000 C CNN
+F 1 "Conn_01x03" V 1200 6850 50  0000 C CNN
+F 2 "Connector_PinHeader_2.54mm:PinHeader_1x03_P2.54mm_Vertical" H 1050 6850 50  0001 C CNN
+F 3 "~" H 1050 6850 50  0001 C CNN
+	1    1050 6850
 	-1   0    0    1
 $EndComp
@@
 L power:+7.5V #PWR0137
 U 1 1 5C591EF9
-P 1200 6750
-F 0 "#PWR0137" H 1200 6600 50  0001 C CNN
-F 1 "+7.5V" V 1215 6878 50  0000 L CNN
-F 2 "" H 1200 6750 50  0001 C CNN
-F 3 "" H 1200 6750 50  0001 C CNN
-	1    1200 6750
+P 1250 6750
+F 0 "#PWR0137" H 1250 6600 50  0001 C CNN
+F 1 "+7.5V" V 1265 6878 50  0000 L CNN
+F 2 "" H 1250 6750 50  0001 C CNN
+F 3 "" H 1250 6750 50  0001 C CNN
+	1    1250 6750
 	0    1    1    0
 $EndComp
@@
 L power:GND #PWR0138
 U 1 1 5C591EFF
-P 1200 6950
-F 0 "#PWR0138" H 1200 6700 50  0001 C CNN
-F 1 "GND" H 1205 6777 50  0000 C CNN
-F 2 "" H 1200 6950 50  0001 C CNN
-F 3 "" H 1200 6950 50  0001 C CNN
-	1    1200 6950
+P 1250 6950
+F 0 "#PWR0138" H 1250 6700 50  0001 C CNN
+F 1 "GND" H 1255 6777 50  0000 C CNN
+F 2 "" H 1250 6950 50  0001 C CNN
+F 3 "" H 1250 6950 50  0001 C CNN
+	1    1250 6950
 	1    0    0    -1
 $EndComp
@@
 	2200 6450 1250 6450
 Wire Wire Line
-	1200 6850 2350 6850
+	1250 6850 2350 6850
 Wire Wire Line
 	2350 6850 2350 4800
 Wire Wire Line
 	2350 4800 2950 4800
-NoConn ~ 2950 4900
 Wire Wire Line
 	3950 4200 4150 4200
@@
 Wire Wire Line
 	4150 4800 3950 4800
-NoConn ~ 3950 4900
 $Comp
 L power:GND #PWR0139
@@
 	1    0    0    -1
 $EndComp
-Wire Wire Line
-	3950 5200 3950 5100
 $Comp
 L power:+7.5V #PWR0142
@@
 	1    0    0    -1
 $EndComp
-Connection ~ 3950 5200
 $Comp
 L 74xx:74HCT244 U101
@@
 Wire Wire Line
 	3650 5900 4150 5900
+Wire Wire Line
+	3950 4900 4150 4900
+$Comp
+L Connector_Generic:Conn_01x03 J110
+U 1 1 5C85B61C
+P 1050 7350
+F 0 "J110" V 1300 7350 50  0000 C CNN
+F 1 "Conn_01x03" V 1200 7350 50  0000 C CNN
+F 2 "Connector_PinHeader_2.54mm:PinHeader_1x03_P2.54mm_Vertical" H 1050 7350 50  0001 C CNN
+F 3 "~" H 1050 7350 50  0001 C CNN
+	1    1050 7350
+	-1   0    0    1
+$EndComp
+$Comp
+L power:+7.5V #PWR0220
+U 1 1 5C86612D
+P 1250 7250
+F 0 "#PWR0220" H 1250 7100 50  0001 C CNN
+F 1 "+7.5V" V 1265 7378 50  0000 L CNN
+F 2 "" H 1250 7250 50  0001 C CNN
+F 3 "" H 1250 7250 50  0001 C CNN
+	1    1250 7250
+	0    1    1    0
+$EndComp
+$Comp
+L power:GND #PWR0221
+U 1 1 5C866164
+P 1250 7450
+F 0 "#PWR0221" H 1250 7200 50  0001 C CNN
+F 1 "GND" H 1255 7277 50  0000 C CNN
+F 2 "" H 1250 7450 50  0001 C CNN
+F 3 "" H 1250 7450 50  0001 C CNN
+	1    1250 7450
+	1    0    0    -1
+$EndComp
+Wire Wire Line
+	2950 4900 2500 4900
+Wire Wire Line
+	2500 4900 2500 7350
+Wire Wire Line
+	2500 7350 1250 7350
 $EndSCHEMATC
