File: motor.sch (KiCad schematic (older format))
At the start: 5 parts

Commit message: Batteries done and raspi added
Connections:
- net VIN renamed +12V
Changed lines of the file:
@@
 $Descr A4 11693 8268
 encoding utf-8
-Sheet 4 7
+Sheet 3 14
 Title ""
 Date ""
@@
 AR Path="/5BE4B1AE" Ref="M?"  Part="1"
 AR Path="/5BE4AF70/5BE4B1AE" Ref="M?"  Part="1"
+AR Path="/5C45D71B/5BE4B1AE" Ref="M?"  Part="1"
+AR Path="/5C45DA60/5BE4B1AE" Ref="M?"  Part="1"
+AR Path="/5C45DEFD/5BE4B1AE" Ref="M?"  Part="1"
+AR Path="/5C45F77E/5BE4B1AE" Ref="M?"  Part="1"
+AR Path="/5C45FA40/5BE4B1AE" Ref="M?"  Part="1"
 F 0 "M?" V 5945 3400 50  0000 C CNN
 F 1 "Motor_DC" V 5854 3400 50  0000 C CNN
@@
 AR Path="/5BE4B1B5" Ref="D?"  Part="1"
 AR Path="/5BE4AF70/5BE4B1B5" Ref="D?"  Part="1"
+AR Path="/5C45D71B/5BE4B1B5" Ref="D?"  Part="1"
+AR Path="/5C45DA60/5BE4B1B5" Ref="D?"  Part="1"
+AR Path="/5C45DEFD/5BE4B1B5" Ref="D?"  Part="1"
+AR Path="/5C45F77E/5BE4B1B5" Ref="D?"  Part="1"
+AR Path="/5C45FA40/5BE4B1B5" Ref="D?"  Part="1"
 F 0 "D?" V 5296 3622 50  0000 R CNN
 F 1 "DIODE" V 5205 3622 50  0000 R CNN
@@
 AR Path="/5BE4B1BC" Ref="D?"  Part="1"
 AR Path="/5BE4AF70/5BE4B1BC" Ref="D?"  Part="1"
+AR Path="/5C45D71B/5BE4B1BC" Ref="D?"  Part="1"
+AR Path="/5C45DA60/5BE4B1BC" Ref="D?"  Part="1"
+AR Path="/5C45DEFD/5BE4B1BC" Ref="D?"  Part="1"
+AR Path="/5C45F77E/5BE4B1BC" Ref="D?"  Part="1"
+AR Path="/5C45FA40/5BE4B1BC" Ref="D?"  Part="1"
 F 0 "D?" V 6196 3622 50  0000 R CNN
 F 1 "DIODE" V 6105 3622 50  0000 R CNN
@@
 AR Path="/5BE4B1C3" Ref="D?"  Part="1"
 AR Path="/5BE4AF70/5BE4B1C3" Ref="D?"  Part="1"
+AR Path="/5C45D71B/5BE4B1C3" Ref="D?"  Part="1"
+AR Path="/5C45DA60/5BE4B1C3" Ref="D?"  Part="1"
+AR Path="/5C45DEFD/5BE4B1C3" Ref="D?"  Part="1"
+AR Path="/5C45F77E/5BE4B1C3" Ref="D?"  Part="1"
+AR Path="/5C45FA40/5BE4B1C3" Ref="D?"  Part="1"
 F 0 "D?" V 6196 2922 50  0000 R CNN
 F 1 "DIODE" V 6105 2922 50  0000 R CNN
@@
 AR Path="/5BE4B1CA" Ref="D?"  Part="1"
 AR Path="/5BE4AF70/5BE4B1CA" Ref="D?"  Part="1"
+AR Path="/5C45D71B/5BE4B1CA" Ref="D?"  Part="1"
+AR Path="/5C45DA60/5BE4B1CA" Ref="D?"  Part="1"
+AR Path="/5C45DEFD/5BE4B1CA" Ref="D?"  Part="1"
+AR Path="/5C45F77E/5BE4B1CA" Ref="D?"  Part="1"
+AR Path="/5C45FA40/5BE4B1CA" Ref="D?"  Part="1"
 F 0 "D?" V 5296 2922 50  0000 R CNN
 F 1 "DIODE" V 5205 2922 50  0000 R CNN
@@
 AR Path="/5BE4B1D2" Ref="#PWR?"  Part="1"
 AR Path="/5BE4AF70/5BE4B1D2" Ref="#PWR?"  Part="1"
+AR Path="/5C45D71B/5BE4B1D2" Ref="#PWR?"  Part="1"
+AR Path="/5C45DA60/5BE4B1D2" Ref="#PWR?"  Part="1"
+AR Path="/5C45DEFD/5BE4B1D2" Ref="#PWR?"  Part="1"
+AR Path="/5C45F77E/5BE4B1D2" Ref="#PWR?"  Part="1"
+AR Path="/5C45FA40/5BE4B1D2" Ref="#PWR?"  Part="1"
 F 0 "#PWR?" H 5250 3700 50  0001 C CNN
 F 1 "GND" H 5255 3777 50  0000 C CNN
@@
 AR Path="/5BE4B1D8" Ref="#PWR?"  Part="1"
 AR Path="/5BE4AF70/5BE4B1D8" Ref="#PWR?"  Part="1"
+AR Path="/5C45D71B/5BE4B1D8" Ref="#PWR?"  Part="1"
+AR Path="/5C45DA60/5BE4B1D8" Ref="#PWR?"  Part="1"
+AR Path="/5C45DEFD/5BE4B1D8" Ref="#PWR?"  Part="1"
+AR Path="/5C45F77E/5BE4B1D8" Ref="#PWR?"  Part="1"
+AR Path="/5C45FA40/5BE4B1D8" Ref="#PWR?"  Part="1"
 F 0 "#PWR?" H 6150 3700 50  0001 C CNN
 F 1 "GND" H 6155 3777 50  0000 C CNN
@@
 Wire Wire Line
 	5250 2850 6150 2850
-Wire Wire Line
-	4800 2850 5250 2850
 Connection ~ 5250 2850
-Text HLabel 4800 2850 0    50   Input ~ 0
-VIN
 Wire Wire Line
 	5100 3450 5250 3450
@@
 Text HLabel 6250 3450 2    50   Input ~ 0
 V2
+$Comp
+L power:+12V #PWR?
+U 1 1 5C45D4C4
+P 5250 2850
+AR Path="/5BE4AF70/5C45D4C4" Ref="#PWR?"  Part="1"
+AR Path="/5C45D71B/5C45D4C4" Ref="#PWR?"  Part="1"
+AR Path="/5C45DA60/5C45D4C4" Ref="#PWR?"  Part="1"
+AR Path="/5C45DEFD/5C45D4C4" Ref="#PWR?"  Part="1"
+AR Path="/5C45F77E/5C45D4C4" Ref="#PWR?"  Part="1"
+AR Path="/5C45FA40/5C45D4C4" Ref="#PWR?"  Part="1"
+F 0 "#PWR?" H 5250 2700 50  0001 C CNN
+F 1 "+12V" H 5265 3023 50  0000 C CNN
+F 2 "" H 5250 2850 50  0001 C CNN
+F 3 "" H 5250 2850 50  0001 C CNN
+	1    5250 2850
+	1    0    0    -1
+$EndComp
 $EndSCHEMATC

Commit message: Schematics Done. Now need to do footprints
Parts:
- gave numbers to parts that had none: 5
Changed lines of the file:
@@
 $Descr A4 11693 8268
 encoding utf-8
-Sheet 3 14
+Sheet 10 14
 Title ""
 Date ""
@@
 P 5650 3450
 AR Path="/5BE4B1AE" Ref="M?"  Part="1"
-AR Path="/5BE4AF70/5BE4B1AE" Ref="M?"  Part="1"
-AR Path="/5C45D71B/5BE4B1AE" Ref="M?"  Part="1"
-AR Path="/5C45DA60/5BE4B1AE" Ref="M?"  Part="1"
-AR Path="/5C45DEFD/5BE4B1AE" Ref="M?"  Part="1"
-AR Path="/5C45F77E/5BE4B1AE" Ref="M?"  Part="1"
-AR Path="/5C45FA40/5BE4B1AE" Ref="M?"  Part="1"
-F 0 "M?" V 5945 3400 50  0000 C CNN
+AR Path="/5BE4AF70/5BE4B1AE" Ref="M301"  Part="1"
+AR Path="/5C45D71B/5BE4B1AE" Ref="M901"  Part="1"
+AR Path="/5C45DA60/5BE4B1AE" Ref="M1001"  Part="1"
+AR Path="/5C45DEFD/5BE4B1AE" Ref="M1101"  Part="1"
+AR Path="/5C45F77E/5BE4B1AE" Ref="M1201"  Part="1"
+AR Path="/5C45FA40/5BE4B1AE" Ref="M1301"  Part="1"
+F 0 "M1301" V 5945 3400 50  0000 C CNN
 F 1 "Motor_DC" V 5854 3400 50  0000 C CNN
 F 2 "" H 5650 3360 50  0001 C CNN
@@
 P 5250 3750
 AR Path="/5BE4B1B5" Ref="D?"  Part="1"
-AR Path="/5BE4AF70/5BE4B1B5" Ref="D?"  Part="1"
-AR Path="/5C45D71B/5BE4B1B5" Ref="D?"  Part="1"
-AR Path="/5C45DA60/5BE4B1B5" Ref="D?"  Part="1"
-AR Path="/5C45DEFD/5BE4B1B5" Ref="D?"  Part="1"
-AR Path="/5C45F77E/5BE4B1B5" Ref="D?"  Part="1"
-AR Path="/5C45FA40/5BE4B1B5" Ref="D?"  Part="1"
-F 0 "D?" V 5296 3622 50  0000 R CNN
+AR Path="/5BE4AF70/5BE4B1B5" Ref="D302"  Part="1"
+AR Path="/5C45D71B/5BE4B1B5" Ref="D902"  Part="1"
+AR Path="/5C45DA60/5BE4B1B5" Ref="D1002"  Part="1"
+AR Path="/5C45DEFD/5BE4B1B5" Ref="D1102"  Part="1"
+AR Path="/5C45F77E/5BE4B1B5" Ref="D1202"  Part="1"
+AR Path="/5C45FA40/5BE4B1B5" Ref="D1302"  Part="1"
+F 0 "D1302" V 5296 3622 50  0000 R CNN
 F 1 "DIODE" V 5205 3622 50  0000 R CNN
 F 2 "" H 5250 3750 50  0001 C CNN
@@
 P 6150 3750
 AR Path="/5BE4B1BC" Ref="D?"  Part="1"
-AR Path="/5BE4AF70/5BE4B1BC" Ref="D?"  Part="1"
-AR Path="/5C45D71B/5BE4B1BC" Ref="D?"  Part="1"
-AR Path="/5C45DA60/5BE4B1BC" Ref="D?"  Part="1"
-AR Path="/5C45DEFD/5BE4B1BC" Ref="D?"  Part="1"
-AR Path="/5C45F77E/5BE4B1BC" Ref="D?"  Part="1"
-AR Path="/5C45FA40/5BE4B1BC" Ref="D?"  Part="1"
-F 0 "D?" V 6196 3622 50  0000 R CNN
+AR Path="/5BE4AF70/5BE4B1BC" Ref="D304"  Part="1"
+AR Path="/5C45D71B/5BE4B1BC" Ref="D904"  Part="1"
+AR Path="/5C45DA60/5BE4B1BC" Ref="D1004"  Part="1"
+AR Path="/5C45DEFD/5BE4B1BC" Ref="D1104"  Part="1"
+AR Path="/5C45F77E/5BE4B1BC" Ref="D1204"  Part="1"
+AR Path="/5C45FA40/5BE4B1BC" Ref="D1304"  Part="1"
+F 0 "D1304" V 6196 3622 50  0000 R CNN
 F 1 "DIODE" V 6105 3622 50  0000 R CNN
 F 2 "" H 6150 3750 50  0001 C CNN
@@
 P 6150 3050
 AR Path="/5BE4B1C3" Ref="D?"  Part="1"
-AR Path="/5BE4AF70/5BE4B1C3" Ref="D?"  Part="1"
-AR Path="/5C45D71B/5BE4B1C3" Ref="D?"  Part="1"
-AR Path="/5C45DA60/5BE4B1C3" Ref="D?"  Part="1"
-AR Path="/5C45DEFD/5BE4B1C3" Ref="D?"  Part="1"
-AR Path="/5C45F77E/5BE4B1C3" Ref="D?"  Part="1"
-AR Path="/5C45FA40/5BE4B1C3" Ref="D?"  Part="1"
-F 0 "D?" V 6196 2922 50  0000 R CNN
+AR Path="/5BE4AF70/5BE4B1C3" Ref="D303"  Part="1"
+AR Path="/5C45D71B/5BE4B1C3" Ref="D903"  Part="1"
+AR Path="/5C45DA60/5BE4B1C3" Ref="D1003"  Part="1"
+AR Path="/5C45DEFD/5BE4B1C3" Ref="D1103"  Part="1"
+AR Path="/5C45F77E/5BE4B1C3" Ref="D1203"  Part="1"
+AR Path="/5C45FA40/5BE4B1C3" Ref="D1303"  Part="1"
+F 0 "D1303" V 6196 2922 50  0000 R CNN
 F 1 "DIODE" V 6105 2922 50  0000 R CNN
 F 2 "" H 6150 3050 50  0001 C CNN
@@
 P 5250 3050
 AR Path="/5BE4B1CA" Ref="D?"  Part="1"
-AR Path="/5BE4AF70/5BE4B1CA" Ref="D?"  Part="1"
-AR Path="/5C45D71B/5BE4B1CA" Ref="D?"  Part="1"
-AR Path="/5C45DA60/5BE4B1CA" Ref="D?"  Part="1"
-AR Path="/5C45DEFD/5BE4B1CA" Ref="D?"  Part="1"
-AR Path="/5C45F77E/5BE4B1CA" Ref="D?"  Part="1"
-AR Path="/5C45FA40/5BE4B1CA" Ref="D?"  Part="1"
-F 0 "D?" V 5296 2922 50  0000 R CNN
+AR Path="/5BE4AF70/5BE4B1CA" Ref="D301"  Part="1"
+AR Path="/5C45D71B/5BE4B1CA" Ref="D901"  Part="1"
+AR Path="/5C45DA60/5BE4B1CA" Ref="D1001"  Part="1"
+AR Path="/5C45DEFD/5BE4B1CA" Ref="D1101"  Part="1"
+AR Path="/5C45F77E/5BE4B1CA" Ref="D1201"  Part="1"
+AR Path="/5C45FA40/5BE4B1CA" Ref="D1301"  Part="1"
+F 0 "D1301" V 5296 2922 50  0000 R CNN
 F 1 "DIODE" V 5205 2922 50  0000 R CNN
 F 2 "" H 5250 3050 50  0001 C CNN
@@
 P 5250 3950
 AR Path="/5BE4B1D2" Ref="#PWR?"  Part="1"
-AR Path="/5BE4AF70/5BE4B1D2" Ref="#PWR?"  Part="1"
-AR Path="/5C45D71B/5BE4B1D2" Ref="#PWR?"  Part="1"
-AR Path="/5C45DA60/5BE4B1D2" Ref="#PWR?"  Part="1"
-AR Path="/5C45DEFD/5BE4B1D2" Ref="#PWR?"  Part="1"
-AR Path="/5C45F77E/5BE4B1D2" Ref="#PWR?"  Part="1"
-AR Path="/5C45FA40/5BE4B1D2" Ref="#PWR?"  Part="1"
-F 0 "#PWR?" H 5250 3700 50  0001 C CNN
+AR Path="/5BE4AF70/5BE4B1D2" Ref="#PWR0124"  Part="1"
+AR Path="/5C45D71B/5BE4B1D2" Ref="#PWR0195"  Part="1"
+AR Path="/5C45DA60/5BE4B1D2" Ref="#PWR0198"  Part="1"
+AR Path="/5C45DEFD/5BE4B1D2" Ref="#PWR0201"  Part="1"
+AR Path="/5C45F77E/5BE4B1D2" Ref="#PWR0204"  Part="1"
+AR Path="/5C45FA40/5BE4B1D2" Ref="#PWR0207"  Part="1"
+F 0 "#PWR0207" H 5250 3700 50  0001 C CNN
 F 1 "GND" H 5255 3777 50  0000 C CNN
 F 2 "" H 5250 3950 50  0001 C CNN
@@
 P 6150 3950
 AR Path="/5BE4B1D8" Ref="#PWR?"  Part="1"
-AR Path="/5BE4AF70/5BE4B1D8" Ref="#PWR?"  Part="1"
-AR Path="/5C45D71B/5BE4B1D8" Ref="#PWR?"  Part="1"
-AR Path="/5C45DA60/5BE4B1D8" Ref="#PWR?"  Part="1"
-AR Path="/5C45DEFD/5BE4B1D8" Ref="#PWR?"  Part="1"
-AR Path="/5C45F77E/5BE4B1D8" Ref="#PWR?"  Part="1"
-AR Path="/5C45FA40/5BE4B1D8" Ref="#PWR?"  Part="1"
-F 0 "#PWR?" H 6150 3700 50  0001 C CNN
+AR Path="/5BE4AF70/5BE4B1D8" Ref="#PWR0125"  Part="1"
+AR Path="/5C45D71B/5BE4B1D8" Ref="#PWR0196"  Part="1"
+AR Path="/5C45DA60/5BE4B1D8" Ref="#PWR0199"  Part="1"
+AR Path="/5C45DEFD/5BE4B1D8" Ref="#PWR0202"  Part="1"
+AR Path="/5C45F77E/5BE4B1D8" Ref="#PWR0205"  Part="1"
+AR Path="/5C45FA40/5BE4B1D8" Ref="#PWR0208"  Part="1"
+F 0 "#PWR0208" H 6150 3700 50  0001 C CNN
 F 1 "GND" H 6155 3777 50  0000 C CNN
 F 2 "" H 6150 3950 50  0001 C CNN
@@
 V2
 $Comp
-L power:+12V #PWR?
+L power:+12V #PWR0126
 U 1 1 5C45D4C4
 P 5250 2850
-AR Path="/5BE4AF70/5C45D4C4" Ref="#PWR?"  Part="1"
-AR Path="/5C45D71B/5C45D4C4" Ref="#PWR?"  Part="1"
-AR Path="/5C45DA60/5C45D4C4" Ref="#PWR?"  Part="1"
-AR Path="/5C45DEFD/5C45D4C4" Ref="#PWR?"  Part="1"
-AR Path="/5C45F77E/5C45D4C4" Ref="#PWR?"  Part="1"
-AR Path="/5C45FA40/5C45D4C4" Ref="#PWR?"  Part="1"
-F 0 "#PWR?" H 5250 2700 50  0001 C CNN
+AR Path="/5BE4AF70/5C45D4C4" Ref="#PWR0126"  Part="1"
+AR Path="/5C45D71B/5C45D4C4" Ref="#PWR0197"  Part="1"
+AR Path="/5C45DA60/5C45D4C4" Ref="#PWR0200"  Part="1"
+AR Path="/5C45DEFD/5C45D4C4" Ref="#PWR0203"  Part="1"
+AR Path="/5C45F77E/5C45D4C4" Ref="#PWR0206"  Part="1"
+AR Path="/5C45FA40/5C45D4C4" Ref="#PWR0209"  Part="1"
+F 0 "#PWR0209" H 5250 2700 50  0001 C CNN
 F 1 "+12V" H 5265 3023 50  0000 C CNN
 F 2 "" H 5250 2850 50  0001 C CNN

Commit message: Schematics done, now assigning footprints to do PCB Next
Parts:
- D301, D302, D303, D304: footprint (none) -> Diode_SMD:D_0805_2012Metric
Changed lines of the file:
@@
 F 0 "D1302" V 5296 3622 50  0000 R CNN
 F 1 "DIODE" V 5205 3622 50  0000 R CNN
-F 2 "" H 5250 3750 50  0001 C CNN
+F 2 "Diode_SMD:D_0805_2012Metric" H 5250 3750 50  0001 C CNN
 F 3 "~" H 5250 3750 50  0001 C CNN
 	1    5250 3750
@@
 F 0 "D1304" V 6196 3622 50  0000 R CNN
 F 1 "DIODE" V 6105 3622 50  0000 R CNN
-F 2 "" H 6150 3750 50  0001 C CNN
+F 2 "Diode_SMD:D_0805_2012Metric" H 6150 3750 50  0001 C CNN
 F 3 "~" H 6150 3750 50  0001 C CNN
 	1    6150 3750
@@
 F 0 "D1303" V 6196 2922 50  0000 R CNN
 F 1 "DIODE" V 6105 2922 50  0000 R CNN
-F 2 "" H 6150 3050 50  0001 C CNN
+F 2 "Diode_SMD:D_0805_2012Metric" H 6150 3050 50  0001 C CNN
 F 3 "~" H 6150 3050 50  0001 C CNN
 	1    6150 3050
@@
 F 0 "D1301" V 5296 2922 50  0000 R CNN
 F 1 "DIODE" V 5205 2922 50  0000 R CNN
-F 2 "" H 5250 3050 50  0001 C CNN
+F 2 "Diode_SMD:D_0805_2012Metric" H 5250 3050 50  0001 C CNN
 F 3 "~" H 5250 3050 50  0001 C CNN
 	1    5250 3050

Commit message: on to pcbs
Parts:
- M301: footprint (none) -> Connector_PinHeader_2.54mm:PinHeader_2x01_P2.54mm_Vertical
Changed lines of the file:
@@
 F 0 "M1301" V 5945 3400 50  0000 C CNN
 F 1 "Motor_DC" V 5854 3400 50  0000 C CNN
-F 2 "" H 5650 3360 50  0001 C CNN
+F 2 "Connector_PinHeader_2.54mm:PinHeader_2x01_P2.54mm_Vertical" H 5650 3360 50  0001 C CNN
 F 3 "~" H 5650 3360 50  0001 C CNN
 	1    5650 3450
