File: H-bridge.sch (KiCad schematic (older format))
At the start: 11 parts, among them U202 L298HN, U401 OP279

Commit message: on to pcbs
Parts:
- U401: footprint (none) -> Package_SO:TSSOP-8_4.4x3mm_P0.65mm
Changed lines of the file:
@@
 F 0 "U201" H 4350 4817 50  0000 C CNN
 F 1 "OP279" H 4350 4726 50  0000 C CNN
-F 2 "" H 4350 4450 50  0001 C CNN
+F 2 "Package_SO:TSSOP-8_4.4x3mm_P0.65mm" H 4350 4450 50  0001 C CNN
 F 3 "http://www.analog.com/media/en/technical-documentation/data-sheets/OP179_279.pdf" H 4350 4450 50  0001 C CNN
 	1    4350 4450
@@
 F 0 "U201" H 4350 5917 50  0000 C CNN
 F 1 "OP279" H 4350 5826 50  0000 C CNN
-F 2 "" H 4350 5550 50  0001 C CNN
+F 2 "Package_SO:TSSOP-8_4.4x3mm_P0.65mm" H 4350 5550 50  0001 C CNN
 F 3 "http://www.analog.com/media/en/technical-documentation/data-sheets/OP179_279.pdf" H 4350 5550 50  0001 C CNN
 	2    4350 5550
@@
 F 0 "U201" H 5558 6396 50  0000 L CNN
 F 1 "OP279" H 5558 6305 50  0000 L CNN
-F 2 "" H 5600 6350 50  0001 C CNN
+F 2 "Package_SO:TSSOP-8_4.4x3mm_P0.65mm" H 5600 6350 50  0001 C CNN
 F 3 "http://www.analog.com/media/en/technical-documentation/data-sheets/OP179_279.pdf" H 5600 6350 50  0001 C CNN
 	3    5600 6350
