File: buck_7v.sch (KiCad schematic (older format))
At the start: 11 parts

Commit message: Schematics Done. Now need to do footprints
Parts:
- R801, R802, R803, R804: renamed from R?; footprint (none) -> Resistor_SMD:R_0805_2012Metric
- gave numbers to parts that had none: 7
Other:
- note added: "TODO: 6V\n"
Changed lines of the file:
@@
 $Descr A4 11693 8268
 encoding utf-8
-Sheet 5 14
+Sheet 8 14
 Title ""
 Date ""
@@
 AR Path="/5BE5CA5D/5BE5CF56" Ref="U?"  Part="1"
 AR Path="/5BE5CC87/5BE5CF56" Ref="U?"  Part="1"
-AR Path="/5C45D160/5BE5CF56" Ref="U?"  Part="1"
-F 0 "U?" H 6275 3915 50  0000 C CNN
+AR Path="/5C45D160/5BE5CF56" Ref="U801"  Part="1"
+F 0 "U801" H 6275 3915 50  0000 C CNN
 F 1 "MP2467" H 6275 3824 50  0000 C CNN
 F 2 "" H 6250 3800 50  0001 C CNN
@@
 AR Path="/5BE5CA5D/5BE5CF5D" Ref="#PWR?"  Part="1"
 AR Path="/5BE5CC87/5BE5CF5D" Ref="#PWR?"  Part="1"
-AR Path="/5C45D160/5BE5CF5D" Ref="#PWR?"  Part="1"
-F 0 "#PWR?" H 4950 3000 50  0001 C CNN
+AR Path="/5C45D160/5BE5CF5D" Ref="#PWR0188"  Part="1"
+F 0 "#PWR0188" H 4950 3000 50  0001 C CNN
 F 1 "GND" H 4955 3077 50  0000 C CNN
 F 2 "" H 4950 3250 50  0001 C CNN
@@
 AR Path="/5BE5CA5D/5BE5CF63" Ref="C?"  Part="1"
 AR Path="/5BE5CC87/5BE5CF63" Ref="C?"  Part="1"
-AR Path="/5C45D160/5BE5CF63" Ref="C?"  Part="1"
-F 0 "C?" V 5098 4050 50  0000 C CNN
+AR Path="/5C45D160/5BE5CF63" Ref="C802"  Part="1"
+F 0 "C802" V 5098 4050 50  0000 C CNN
 F 1 "C" V 5189 4050 50  0000 C CNN
 F 2 "" H 5388 3900 50  0001 C CNN
@@
 AR Path="/5BE5CA5D/5BE5CF6E" Ref="C?"  Part="1"
 AR Path="/5BE5CC87/5BE5CF6E" Ref="C?"  Part="1"
-AR Path="/5C45D160/5BE5CF6E" Ref="C?"  Part="1"
-F 0 "C?" H 4665 3746 50  0000 L CNN
+AR Path="/5C45D160/5BE5CF6E" Ref="C801"  Part="1"
+F 0 "C801" H 4665 3746 50  0000 L CNN
 F 1 "C" H 4665 3655 50  0000 L CNN
 F 2 "" H 4588 3550 50  0001 C CNN
@@
 AR Path="/5BE5CA5D/5BE5CF75" Ref="#PWR?"  Part="1"
 AR Path="/5BE5CC87/5BE5CF75" Ref="#PWR?"  Part="1"
-AR Path="/5C45D160/5BE5CF75" Ref="#PWR?"  Part="1"
-F 0 "#PWR?" H 4550 3600 50  0001 C CNN
+AR Path="/5C45D160/5BE5CF75" Ref="#PWR0189"  Part="1"
+F 0 "#PWR0189" H 4550 3600 50  0001 C CNN
 F 1 "GND" H 4555 3677 50  0000 C CNN
 F 2 "" H 4550 3850 50  0001 C CNN
@@
 AR Path="/5BE5CA5D/5BE5CF7C" Ref="C?"  Part="1"
 AR Path="/5BE5CC87/5BE5CF7C" Ref="C?"  Part="1"
-AR Path="/5C45D160/5BE5CF7C" Ref="C?"  Part="1"
-F 0 "C?" V 5598 3450 50  0000 C CNN
+AR Path="/5C45D160/5BE5CF7C" Ref="C803"  Part="1"
+F 0 "C803" V 5598 3450 50  0000 C CNN
 F 1 "220pF" V 5689 3450 50  0000 C CNN
 F 2 "" H 5888 3300 50  0001 C CNN
@@
 AR Path="/5BE5CA5D/5BE5CF83" Ref="R?"  Part="1"
 AR Path="/5BE5CC87/5BE5CF83" Ref="R?"  Part="1"
-AR Path="/5C45D160/5BE5CF83" Ref="R?"  Part="1"
-F 0 "R?" V 5943 3450 50  0000 C CNN
+AR Path="/5C45D160/5BE5CF83" Ref="R802"  Part="1"
+F 0 "R802" V 5943 3450 50  0000 C CNN
 F 1 "68k" V 6034 3450 50  0000 C CNN
-F 2 "" V 6080 3450 50  0001 C CNN
+F 2 "Resistor_SMD:R_0805_2012Metric" V 6080 3450 50  0001 C CNN
 F 3 "~" H 6150 3450 50  0001 C CNN
 	1    6150 3450
@@
 AR Path="/5BE5CA5D/5BE5CF8A" Ref="#PWR?"  Part="1"
 AR Path="/5BE5CC87/5BE5CF8A" Ref="#PWR?"  Part="1"
-AR Path="/5C45D160/5BE5CF8A" Ref="#PWR?"  Part="1"
-F 0 "#PWR?" H 6400 3200 50  0001 C CNN
+AR Path="/5C45D160/5BE5CF8A" Ref="#PWR0190"  Part="1"
+F 0 "#PWR0190" H 6400 3200 50  0001 C CNN
 F 1 "GND" H 6405 3277 50  0000 C CNN
 F 2 "" H 6400 3450 50  0001 C CNN
 F 3 "" H 6400 3450 50  0001 C CNN
 	1    6400 3450
-	-1   0    0    1
+	1    0    0    -1
 $EndComp
 Wire Wire Line
@@
 AR Path="/5BE5CA5D/5BE5CF91" Ref="R?"  Part="1"
 AR Path="/5BE5CC87/5BE5CF91" Ref="R?"  Part="1"
-AR Path="/5C45D160/5BE5CF91" Ref="R?"  Part="1"
-F 0 "R?" H 4680 3254 50  0000 R CNN
+AR Path="/5C45D160/5BE5CF91" Ref="R801"  Part="1"
+F 0 "R801" H 4680 3254 50  0000 R CNN
 F 1 "200k" H 4680 3345 50  0000 R CNN
-F 2 "" V 4680 3300 50  0001 C CNN
+F 2 "Resistor_SMD:R_0805_2012Metric" V 4680 3300 50  0001 C CNN
 F 3 "~" H 4750 3300 50  0001 C CNN
 	1    4750 3300
@@
 AR Path="/5BE5CA5D/5BE5CF99" Ref="#PWR?"  Part="1"
 AR Path="/5BE5CC87/5BE5CF99" Ref="#PWR?"  Part="1"
-AR Path="/5C45D160/5BE5CF99" Ref="#PWR?"  Part="1"
-F 0 "#PWR?" H 4750 2900 50  0001 C CNN
+AR Path="/5C45D160/5BE5CF99" Ref="#PWR0191"  Part="1"
+F 0 "#PWR0191" H 4750 2900 50  0001 C CNN
 F 1 "GND" H 4755 2977 50  0000 C CNN
 F 2 "" H 4750 3150 50  0001 C CNN
@@
 AR Path="/5BE5CA5D/5BE5CFA0" Ref="D?"  Part="1"
 AR Path="/5BE5CC87/5BE5CFA0" Ref="D?"  Part="1"
-AR Path="/5C45D160/5BE5CFA0" Ref="D?"  Part="1"
-F 0 "D?" V 5654 4279 50  0000 L CNN
+AR Path="/5C45D160/5BE5CFA0" Ref="D801"  Part="1"
+F 0 "D801" V 5654 4279 50  0000 L CNN
 F 1 "D_Schottky" V 5745 4279 50  0000 L CNN
 F 2 "" H 5700 4200 50  0001 C CNN
@@
 AR Path="/5BE5CA5D/5BE5CFA8" Ref="#PWR?"  Part="1"
 AR Path="/5BE5CC87/5BE5CFA8" Ref="#PWR?"  Part="1"
-AR Path="/5C45D160/5BE5CFA8" Ref="#PWR?"  Part="1"
-F 0 "#PWR?" H 5700 4100 50  0001 C CNN
+AR Path="/5C45D160/5BE5CFA8" Ref="#PWR0192"  Part="1"
+F 0 "#PWR0192" H 5700 4100 50  0001 C CNN
 F 1 "GND" H 5705 4177 50  0000 C CNN
 F 2 "" H 5700 4350 50  0001 C CNN
@@
 AR Path="/5BE5CA5D/5BE5CFAE" Ref="L?"  Part="1"
 AR Path="/5BE5CC87/5BE5CFAE" Ref="L?"  Part="1"
-AR Path="/5C45D160/5BE5CFAE" Ref="L?"  Part="1"
-F 0 "L?" V 6290 4050 50  0000 C CNN
+AR Path="/5C45D160/5BE5CFAE" Ref="L801"  Part="1"
+F 0 "L801" V 6290 4050 50  0000 C CNN
 F 1 "L" V 6199 4050 50  0000 C CNN
 F 2 "" H 6100 4050 50  0001 C CNN
@@
 AR Path="/5BE5CA5D/5BE5CFB6" Ref="C?"  Part="1"
 AR Path="/5BE5CC87/5BE5CFB6" Ref="C?"  Part="1"
-AR Path="/5C45D160/5BE5CFB6" Ref="C?"  Part="1"
-F 0 "C?" H 6515 4246 50  0000 L CNN
+AR Path="/5C45D160/5BE5CFB6" Ref="C804"  Part="1"
+F 0 "C804" H 6515 4246 50  0000 L CNN
 F 1 "220pF" H 6515 4155 50  0000 L CNN
 F 2 "" H 6438 4050 50  0001 C CNN
@@
 AR Path="/5BE5CA5D/5BE5CFBD" Ref="#PWR?"  Part="1"
 AR Path="/5BE5CC87/5BE5CFBD" Ref="#PWR?"  Part="1"
-AR Path="/5C45D160/5BE5CFBD" Ref="#PWR?"  Part="1"
-F 0 "#PWR?" H 6400 4100 50  0001 C CNN
+AR Path="/5C45D160/5BE5CFBD" Ref="#PWR0193"  Part="1"
+F 0 "#PWR0193" H 6400 4100 50  0001 C CNN
 F 1 "GND" H 6405 4177 50  0000 C CNN
 F 2 "" H 6400 4350 50  0001 C CNN
@@
 AR Path="/5BE5CA5D/5BE5CFC3" Ref="R?"  Part="1"
 AR Path="/5BE5CC87/5BE5CFC3" Ref="R?"  Part="1"
-AR Path="/5C45D160/5BE5CFC3" Ref="R?"  Part="1"
-F 0 "R?" H 6770 3746 50  0000 L CNN
+AR Path="/5C45D160/5BE5CFC3" Ref="R804"  Part="1"
+F 0 "R804" H 6770 3746 50  0000 L CNN
 F 1 "75k" H 6770 3655 50  0000 L CNN
-F 2 "" V 6630 3700 50  0001 C CNN
+F 2 "Resistor_SMD:R_0805_2012Metric" V 6630 3700 50  0001 C CNN
 F 3 "~" H 6700 3700 50  0001 C CNN
 	1    6700 3700
@@
 AR Path="/5BE5CA5D/5BE5CFCA" Ref="R?"  Part="1"
 AR Path="/5BE5CC87/5BE5CFCA" Ref="R?"  Part="1"
-AR Path="/5C45D160/5BE5CFCA" Ref="R?"  Part="1"
-F 0 "R?" H 6770 3096 50  0000 L CNN
+AR Path="/5C45D160/5BE5CFCA" Ref="R803"  Part="1"
+F 0 "R803" H 6770 3096 50  0000 L CNN
 F 1 "10k" H 6770 3005 50  0000 L CNN
-F 2 "" V 6630 3050 50  0001 C CNN
+F 2 "Resistor_SMD:R_0805_2012Metric" V 6630 3050 50  0001 C CNN
 F 3 "~" H 6700 3050 50  0001 C CNN
 	1    6700 3050
@@
 AR Path="/5BE5CA5D/5BE5CFD6" Ref="#PWR?"  Part="1"
 AR Path="/5BE5CC87/5BE5CFD6" Ref="#PWR?"  Part="1"
-AR Path="/5C45D160/5BE5CFD6" Ref="#PWR?"  Part="1"
-F 0 "#PWR?" H 6700 2650 50  0001 C CNN
+AR Path="/5C45D160/5BE5CFD6" Ref="#PWR0194"  Part="1"
+F 0 "#PWR0194" H 6700 2650 50  0001 C CNN
 F 1 "GND" H 6705 2727 50  0000 C CNN
 F 2 "" H 6700 2900 50  0001 C CNN
@@
 Wire Wire Line
 	6250 4050 6400 4050
+Text Notes 7000 3350 0    50   ~ 0
+TODO: 6V\n
 $EndSCHEMATC

Commit message: Schematics done, now assigning footprints to do PCB Next
Parts:
- C801, C802, C803, C804: footprint (none) -> Capacitor_SMD:C_0805_2012Metric
- D801: footprint (none) -> Diode_SMD:D_0805_2012Metric
- L801: footprint (none) -> Inductor_SMD:L_0805_2012Metric
Changed lines of the file:
@@
 F 0 "C802" V 5098 4050 50  0000 C CNN
 F 1 "C" V 5189 4050 50  0000 C CNN
-F 2 "" H 5388 3900 50  0001 C CNN
+F 2 "Capacitor_SMD:C_0805_2012Metric" H 5388 3900 50  0001 C CNN
 F 3 "~" H 5350 4050 50  0001 C CNN
 	1    5350 4050
@@
 F 0 "C801" H 4665 3746 50  0000 L CNN
 F 1 "C" H 4665 3655 50  0000 L CNN
-F 2 "" H 4588 3550 50  0001 C CNN
+F 2 "Capacitor_SMD:C_0805_2012Metric" H 4588 3550 50  0001 C CNN
 F 3 "~" H 4550 3700 50  0001 C CNN
 	1    4550 3700
@@
 F 0 "C803" V 5598 3450 50  0000 C CNN
 F 1 "220pF" V 5689 3450 50  0000 C CNN
-F 2 "" H 5888 3300 50  0001 C CNN
+F 2 "Capacitor_SMD:C_0805_2012Metric" H 5888 3300 50  0001 C CNN
 F 3 "~" H 5850 3450 50  0001 C CNN
 	1    5850 3450
@@
 F 0 "D801" V 5654 4279 50  0000 L CNN
 F 1 "D_Schottky" V 5745 4279 50  0000 L CNN
-F 2 "" H 5700 4200 50  0001 C CNN
+F 2 "Diode_SMD:D_0805_2012Metric" H 5700 4200 50  0001 C CNN
 F 3 "~" H 5700 4200 50  0001 C CNN
 	1    5700 4200
@@
 F 0 "L801" V 6290 4050 50  0000 C CNN
 F 1 "L" V 6199 4050 50  0000 C CNN
-F 2 "" H 6100 4050 50  0001 C CNN
+F 2 "Inductor_SMD:L_0805_2012Metric" H 6100 4050 50  0001 C CNN
 F 3 "~" H 6100 4050 50  0001 C CNN
 	1    6100 4050
@@
 F 0 "C804" H 6515 4246 50  0000 L CNN
 F 1 "220pF" H 6515 4155 50  0000 L CNN
-F 2 "" H 6438 4050 50  0001 C CNN
+F 2 "Capacitor_SMD:C_0805_2012Metric" H 6438 4050 50  0001 C CNN
 F 3 "~" H 6400 4200 50  0001 C CNN
 	1    6400 4200

Commit message: on to pcbs
Parts:
- U801: footprint (none) -> Package_SO:SOIC-8_3.9x4.9mm_P1.27mm
Changed lines of the file:
@@
 F 0 "U801" H 6275 3915 50  0000 C CNN
 F 1 "MP2467" H 6275 3824 50  0000 C CNN
-F 2 "" H 6250 3800 50  0001 C CNN
+F 2 "Package_SO:SOIC-8_3.9x4.9mm_P1.27mm" H 6250 3800 50  0001 C CNN
 F 3 "" H 6250 3800 50  0001 C CNN
 	1    5800 4250

Commit message: updated layout
Parts:
- U801: symbol Converter_ACDC:MP2467 -> Mars-Rover-rescue:MP2467-Converter_ACDC
Changed lines of the file:
@@
 $EndDescr
 $Comp
-L Converter_ACDC:MP2467 U?
+L Mars-Rover-rescue:MP2467-Converter_ACDC U?
 U 1 1 5BE5CF56
 P 5800 4250
